File: Kicad files/OpenRover/OpenRover.kicad_sch (KiCad schematic)
At the start: 0 parts

Commit message: Updated with Allan his work.
Parts:
- added C1, C10, C11, C12, C13, C14, C2, C3, C4, C5, C6, C7, C8, C9: 0.1, symbol Device:C
- added C15, C18, C19: 1uF, symbol Device:C
- added C16: 1nF, symbol Device:C
- added C17: 10uF, symbol Device:C
- added D1, D2, D3, D4, D5, D6, D7: BAV23, Package_TO_SOT_SMD:SOT-23, symbol Diode:BAV99
- added D8, D9: 1N4148W, Diode_SMD:D_SOD-123, symbol Diode:1N4148W
- added FB1, FB2: Ferrite_Bead, symbol Device:Ferrite_Bead
- added L1: 2.2uH, IND_TAIYO_NRS6020_TAY, symbol 2021-01-06_02-33-04:NRS6020T2R2NMGJ
- added Q1: FQT7N10L, Package_TO_SOT_SMD:SOT-23, symbol Transistor_FET:IRLML6402
- added Q2: BC846, Package_TO_SOT_SMD:SOT-23, symbol Transistor_BJT:BC846
- added Q3: MMDT3906, Package_TO_SOT_SMD:SOT-363_SC-70-6, symbol Transistor_BJT:MMDT3906
- added R1, R2, R3, R4: 22M, symbol Device:R
- added R10, R15: R, symbol Device:R
- added R11: 121k, symbol Device:R
- added R12: 33k, symbol Device:R
- added R13: 100, symbol Device:R
- added R14: 100k, symbol Device:R
- added R5: 3.16M, symbol Device:R
- added R6: 560K, symbol Device:R
- added R7: 4M7, symbol Device:R
- added R8, R9: 100K, symbol Device:R
- added U1: 74HC14, symbol 74xx:74HC14
- added U2: MAX4162, Package_TO_SOT_SMD:SOT-23-5, symbol Amplifier_Operational:TLV2371DBV
- added U3: CD14538BM, symbol 4xxx:4538
- added U4: MAX6008AEUR+T, Package_TO_SOT_SMD:SOT-23, symbol Reference_Voltage:MAX6035xxUR30
Connections:
- new net: C14.1, R8.1, R9.1, U1.1
- new net: D8.1 (K), U1.11, U1.13, U1.2, U1.3, U1.5, U1.9
- new net: Q1.1 (G), U1.10, U1.12, U1.4, U1.6, U1.8
- new net: C15.1, R10.1, U1.14 (VCC)
- new net: C2.2, C4.1, D1.2 (A), D2.1 (K)
- new net: C4.2, C6.1, D2.2 (A), D3.1 (K)
- new net: C3.2, C5.1, D2.3 (K)
- new net: C6.2, C8.1, D3.2 (A), D4.1 (K)
- new net: C5.2, C7.1, D3.3 (K)
- new net: C10.1, C8.2, D4.2 (A), D5.1 (K)
- new net: C7.2, C9.1, D4.3 (K)
- new net: C10.2, C12.1, D5.2 (A), D6.1 (K)
- new net: C11.1, C9.2, D5.3 (K)
- new net: C12.2, D6.2 (A), D7.1 (K)
- new net: C11.2, C13.1, D6.3 (K)
- new net: C1.2, C3.1, D1.3 (K), R1.1
- new net: C13.2, D7.3 (K), R7.1
- new net: R8.2, U2.1
- new net: R6.2, U2.3 (+), U4.1 (IN)
- new net: R4.1, R5.1, U2.4 (-)
- new net: C18.1, FB1.2, L1.1
- new net: C19.1, R11.1, R13.2, U3.12 (Clk+), U3.16 (VDD), U3.3 (R)
- new net: C16.1, R11.2, U3.2 (RxCx)
- new net: R1.2, R2.2
- new net: R2.1, R3.2
- new net: R3.1, R4.2
- new net: D9.1 (K), R12.1, U3.5 (Clk-)
- new net: D9.2 (A), U3.6 (Q)
- new net: FB2.2, R10.2
- new net: D8.2 (A), R9.2
- new net: Q3.1 (E1), Q3.4 (E2), R15.2
- new net: Q2.1 (B), Q3.6 (C1)
- new net: Q2.3 (C), R12.2, R14.2
- new net: R14.1, R15.1
- new net +3V3: C17.1, FB1.1, FB2.1, R13.1, R6.1
- new net GND: C1.1, C14.2, C15.2, C16.2, C17.2, C18.2, C19.2, C2.1, D1.1 (K), L1.2, Q1.2 (S), Q1.3 (D), Q2.2 (E), Q3.3 (C2), R5.2, U1.7 (GND), U2.2 (V-), U3.1 (VSS), U3.11 (Clk-), U3.13 (R), U3.15 (VSS), U3.4 (Clk+), U3.8 (VSS), U4.2 (OUT)
Other:
- company: (none) -> SafeCast
- title: (none) -> OpenRover
