File: Kicad files/OpenRover/OpenRover.kicad_sch (KiCad schematic)
At the start: 53 parts, among them Q1 FQT7N10L, Q2 BC846, Q3 MMDT3906, U1 74HC14, U2 MAX4162, U3 CD14538BM, U4 MAX6008AEUR+T

Commit message: Tested 74HC14 adding to the footprints
Parts:
- U1: footprint (none) -> Package_SO:SOIC-14_3.9x8.7mm_P1.27mm
Changed lines of the file:
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@@
     (property "Reference" "U1" (id 0) (at 63.5 82.1182 0))
     (property "Value" "74HC14" (id 1) (at 63.5 84.4296 0))
-    (property "Footprint" "" (id 2) (at 63.5 90.17 0)
+    (property "Footprint" "Package_SO:SOIC-14_3.9x8.7mm_P1.27mm" (id 2) (at 63.5 90.17 0)
       (effects (font (size 1.27 1.27)) hide)
     )
@@
     (property "Reference" "U1" (id 0) (at 88.9 47.8282 0))
     (property "Value" "74HC14" (id 1) (at 88.9 50.1396 0))
-    (property "Footprint" "" (id 2) (at 88.9 55.88 0)
+    (property "Footprint" "Package_SO:SOIC-14_3.9x8.7mm_P1.27mm" (id 2) (at 88.9 55.88 0)
       (effects (font (size 1.27 1.27)) hide)
     )
@@
     (property "Reference" "U1" (id 0) (at 88.9 65.6082 0))
     (property "Value" "74HC14" (id 1) (at 88.9 67.9196 0))
-    (property "Footprint" "" (id 2) (at 88.9 73.66 0)
+    (property "Footprint" "Package_SO:SOIC-14_3.9x8.7mm_P1.27mm" (id 2) (at 88.9 73.66 0)
       (effects (font (size 1.27 1.27)) hide)
     )
@@
     (property "Reference" "U1" (id 0) (at 88.9 82.1182 0))
     (property "Value" "74HC14" (id 1) (at 88.9 84.4296 0))
-    (property "Footprint" "" (id 2) (at 88.9 90.17 0)
+    (property "Footprint" "Package_SO:SOIC-14_3.9x8.7mm_P1.27mm" (id 2) (at 88.9 90.17 0)
       (effects (font (size 1.27 1.27)) hide)
     )
@@
     (property "Reference" "U1" (id 0) (at 88.9 99.8982 0))
     (property "Value" "74HC14" (id 1) (at 88.9 102.2096 0))
-    (property "Footprint" "" (id 2) (at 88.9 107.95 0)
+    (property "Footprint" "Package_SO:SOIC-14_3.9x8.7mm_P1.27mm" (id 2) (at 88.9 107.95 0)
       (effects (font (size 1.27 1.27)) hide)
     )
@@
     (property "Reference" "U1" (id 0) (at 88.9 116.4082 0))
     (property "Value" "74HC14" (id 1) (at 88.9 118.7196 0))
-    (property "Footprint" "" (id 2) (at 88.9 124.46 0)
+    (property "Footprint" "Package_SO:SOIC-14_3.9x8.7mm_P1.27mm" (id 2) (at 88.9 124.46 0)
       (effects (font (size 1.27 1.27)) hide)
     )
@@
       (effects (font (size 1.27 1.27)) (justify left))
     )
-    (property "Footprint" "" (id 2) (at 30.48 54.61 0)
+    (property "Footprint" "Package_SO:SOIC-14_3.9x8.7mm_P1.27mm" (id 2) (at 30.48 54.61 0)
       (effects (font (size 1.27 1.27)) hide)
     )
@@
     )
     (path "/00000000-0000-0000-0000-00005ff4e574"
-      (reference "U1") (unit 1) (value "74HC14") (footprint "")
+      (reference "U1") (unit 1) (value "74HC14") (footprint "Package_SO:SOIC-14_3.9x8.7mm_P1.27mm")
     )
     (path "/00000000-0000-0000-0000-00005ff4f0bc"
-      (reference "U1") (unit 2) (value "74HC14") (footprint "")
+      (reference "U1") (unit 2) (value "74HC14") (footprint "Package_SO:SOIC-14_3.9x8.7mm_P1.27mm")
     )
     (path "/00000000-0000-0000-0000-00005ff4ffd6"
-      (reference "U1") (unit 3) (value "74HC14") (footprint "")
+      (reference "U1") (unit 3) (value "74HC14") (footprint "Package_SO:SOIC-14_3.9x8.7mm_P1.27mm")
     )
     (path "/00000000-0000-0000-0000-00005ff512ab"
-      (reference "U1") (unit 4) (value "74HC14") (footprint "")
+      (reference "U1") (unit 4) (value "74HC14") (footprint "Package_SO:SOIC-14_3.9x8.7mm_P1.27mm")
     )
     (path "/00000000-0000-0000-0000-00005ff52243"
-      (reference "U1") (unit 5) (value "74HC14") (footprint "")
+      (reference "U1") (unit 5) (value "74HC14") (footprint "Package_SO:SOIC-14_3.9x8.7mm_P1.27mm")
     )
     (path "/00000000-0000-0000-0000-00005ff531e2"
-      (reference "U1") (unit 6) (value "74HC14") (footprint "")
+      (reference "U1") (unit 6) (value "74HC14") (footprint "Package_SO:SOIC-14_3.9x8.7mm_P1.27mm")
     )
     (path "/00000000-0000-0000-0000-00005ff54255"
-      (reference "U1") (unit 7) (value "74HC14") (footprint "")
+      (reference "U1") (unit 7) (value "74HC14") (footprint "Package_SO:SOIC-14_3.9x8.7mm_P1.27mm")
     )
     (path "/00000000-0000-0000-0000-00005ff98bd3"

Commit message: Updated the files from the allan zip files.
Parts:
- removed Q1: FQT7N10L, Package_TO_SOT_SMD:SOT-23, symbol Transistor_FET:IRLML6402
- added C20, C21, C22: C, Capacitor_SMD:C_0805_2012Metric, symbol Device:C
- added J1: Conn_01x03_Male, Connector_PinHeader_2.54mm:PinHeader_1x03_P2.54mm_Vertical, symbol Connector:Conn_01x03_Male
- added Q1: FQT7N10, Package_TO_SOT_SMD:SOT-223-3_TabPin2, symbol Transistor_FET:IRF6655
- added R16: 392k, Resistor_SMD:R_0805_2012Metric, symbol Device:R
- added R17: 1M, Resistor_SMD:R_0805_2012Metric, symbol Device:R
- added R18: 499k, Resistor_SMD:R_0805_2012Metric, symbol Device:R
- added R19: 1k, Resistor_SMD:R_0805_2012Metric, symbol Device:R
- added R20: 100k, Resistor_SMD:R_0805_2012Metric, symbol Device:R
- added R21: 47k, Resistor_SMD:R_0805_2012Metric, symbol Device:R
- added R22: 20k, Resistor_SMD:R_0805_2012Metric, symbol Device:R
- C1, C10, C11, C12, C13, C2, C3, C4, C5, C6, C7, C8, C9, FB1, FB2, R1, R10, R11, R12, R13, R14, R2, R3, R4, R5, R6, R8, R9: footprint (none) -> Resistor_SMD:R_0805_2012Metric
- C14, C15, C16, C18, C19: footprint (none) -> Capacitor_SMD:C_0805_2012Metric
- C17: footprint (none) -> Capacitor_SMD:C_1210_3225Metric
- L1: footprint IND_TAIYO_NRS6020_TAY -> Inductor_SMD:L_Taiyo-Yuden_MD-4040
- R15: value R -> 1M49; footprint (none) -> Resistor_SMD:R_0805_2012Metric
- R7: footprint (none) -> Resistor_SMD:R_1206_3216Metric
- U3: footprint (none) -> Package_SO:SOIC-16_3.9x9.9mm_P1.27mm
Connections:
- net +3V3: now also J1.1 (Pin_1), R19.2
- net GND: now also C20.2, C21.2, C22.2, J1.3 (Pin_3), Q1.3 (S), R16.2, R17.2, R22.2; no longer C2.1, D1.1 (K), L1.2
- net at U1.10, U1.12, U1.4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: now also Q1.2 (G)
- net +2V5: now reaches R6.2, U2.3 (+), U4.1 (IN)
- net +2V5: now also R15.1
- net at D9.2 (A), U3.6 (Q): now also J1.2 (Pin_2)
- net at Q3.1 (E1), Q3.4 (E2): now also R18.2; no longer R15.2
- net at Q3.2 (B1): now also R15.2, C20.1, R16.1
- net at Q2.1 (B), Q3.6 (C1): now also R17.1
- net at Q3.5 (B2): now also R20.1
- net at R14.1: now also C21.1, R18.1, R19.1; no longer R15.1
- new net: C2.1, D1.1 (K), L1.2, Q1.1 (D)
- new net: C22.1, R20.2, R21.2, R22.1
Other:
- moved on the sheet: Q2, Q3A, Q3B
