File: Kicad files/OpenHVPS-2/_autosave-OpenHVPS-2.kicad_pcb (KiCad board)
At the start: 2 copper layers, 45 x 20.5 mm, 69 parts, among them J1 Conn_01x03_Male, J2 Conn_01x03_Male, Q1 FQT7N10, Q2 BC846, Q3 MMDT3906, U1 MAX6008AEUR+T, U2 74HC14, U3 MAX4162, U4 CD14538BM

Commit message: layout chnages
Parts:
- H2: footprint TestPoint:TestPoint_Loop_D3.80mm_Drill2.0mm -> TestPoint:TestPoint_Loop_D2.60mm_Drill1.4mm_Beaded
- moved C2 0.92 mm to (138.4, 71.1)
- moved FB1 0.92 mm to (130.8, 71.1)
- moved R5 0.92 mm to (134.4, 71.1)
- moved H1 0.59 mm to (138.4, 75.2)
- moved U3 0.26 mm to (156.5, 74.9)
Changed lines of the file:
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@@
     )
   )
-  (footprint "TestPoint:TestPoint_Loop_D3.80mm_Drill2.0mm" (layer "F.Cu")
+  (footprint "TestPoint:TestPoint_Loop_D2.60mm_Drill1.4mm_Beaded" (layer "F.Cu")
     (at 163 70 90)
-    (descr "wire loop as test point, loop diameter 3.8mm, hole diameter 2.0mm")
+    (descr "wire loop with bead as test point, loop diameter2.6mm, hole diameter 1.4mm")
     (tags "test point wire loop bead")
     (property "Sheet file" "OpenHVPS-2.kicad_sch")
     (property "Sheet name" "")
     (attr through_hole)
-    (fp_text reference "H2" (at 0.5 2.8 90) (layer "F.SilkS")
+    (fp_text reference "H2" (at 0.7 2.5 90) (layer "F.SilkS")
       (effects (font (size 1 1) (thickness 0.15)))
     )
-    (fp_text value "Anode" (at -2.898 0.322 180) (layer "F.Fab")
+    (fp_text value "Anode" (at 0 -2.8 90) (layer "F.Fab")
       (effects (font (size 1 1) (thickness 0.15)))
     )
-    (fp_text user "${REFERENCE}" (at 0.5 2.8 90) (layer "F.Fab")
+    (fp_text user "${REFERENCE}" (at 0.7 2.5 90) (layer "F.Fab")
       (effects (font (size 1 1) (thickness 0.15)))
     )
-    (fp_circle (center 0 0) (end 2.1 0) (layer "F.SilkS") (width 0.12) (fill none))
-    (fp_circle (center 0 0) (end 2.3 0) (layer "F.CrtYd") (width 0.05) (fill none))
-    (fp_line (start 1.9 -0.3) (end -1.9 -0.3) (layer "F.Fab") (width 0.12))
-    (fp_line (start 1.9 0.3) (end 1.9 -0.3) (layer "F.Fab") (width 0.12))
-    (fp_line (start -1.9 0.3) (end 1.9 0.3) (layer "F.Fab") (width 0.12))
-    (fp_line (start -1.9 -0.3) (end -1.9 0.3) (layer "F.Fab") (width 0.12))
-    (pad "1" thru_hole circle (at 0 0 90) (locked) (size 3.6 3.6) (drill 2) (layers *.Cu *.Mask)
+    (fp_circle (center 0 0) (end 1.7 0) (layer "F.SilkS") (width 0.12) (fill none))
+    (fp_circle (center 0 0) (end 2 0) (layer "F.CrtYd") (width 0.05) (fill none))
+    (fp_line (start 1.3 -0.3) (end -1.3 -0.3) (layer "F.Fab") (width 0.12))
+    (fp_line (start -1.3 -0.3) (end -1.3 0.3) (layer "F.Fab") (width 0.12))
+    (fp_line (start -1.3 0.3) (end 1.3 0.3) (layer "F.Fab") (width 0.12))
+    (fp_line (start 1.3 0.3) (end 1.3 -0.3) (layer "F.Fab") (width 0.12))
+    (fp_circle (center 0 0) (end 1.5 0) (layer "F.Fab") (width 0.12) (fill none))
+    (pad "1" thru_hole circle (at 0 0 90) (locked) (size 2.8 2.8) (drill 1.4) (layers *.Cu *.Mask)
       (net 41 "Net-(R1-Pad2)") (pinfunction "1"))
-    (model "${KICAD6_3DMODEL_DIR}/TestPoint.3dshapes/TestPoint_Loop_D3.80mm_Drill2.0mm.wrl"
+    (model "${KICAD6_3DMODEL_DIR}/TestPoint.3dshapes/TestPoint_Loop_D2.60mm_Drill1.4mm_Beaded.wrl"
       (offset (xyz 0 0 0))
       (scale (xyz 1 1 1))
@@
   )
   (footprint "Capacitor_SMD:C_0805_2012Metric" (layer "F.Cu")
-    (at 139.126 70.612 180)
+    (at 138.364 71.12 180)
     (descr "Capacitor SMD 0805 (2012 Metric), square (rectangular) end terminal, IPC_7351 nominal, (Body size source: IPC-SM-782 page 76, https://www.pcb-3d.com/wordpress/wp-content/uploads/ipc-sm-782a_amendment_1_and_2.pdf, https://docs.google.com/spreadsheets/d/1BsfQQcO9C6DZCsRaXUlFlo91Tg2WpOkGARC1WS5S8t0/edit?usp=sharing), generated with kicad-footprint-generator")
     (tags "capacitor")
@@
   )
   (footprint "Resistor_SMD:R_0805_2012Metric" (layer "F.Cu")
-    (at 135.128 70.612)
+    (at 134.366 71.12)
     (descr "Resistor SMD 0805 (2012 Metric), square (rectangular) end terminal, IPC_7351 nominal, (Body size source: IPC-SM-782 page 72, https://www.pcb-3d.com/wordpress/wp-content/uploads/ipc-sm-782a_amendment_1_and_2.pdf), generated with kicad-footprint-generator")
     (tags "resistor")
@@
   )
   (footprint "TestPoint:TestPoint_Loop_D2.60mm_Drill1.4mm_Beaded" (layer "F.Cu")
-    (at 138.938 74.93)
+    (at 138.43 75.23)
     (descr "wire loop with bead as test point, loop diameter2.6mm, hole diameter 1.4mm")
     (tags "test point wire loop bead")
@@
       (effects (font (size 1 1) (thickness 0.15)))
     )
-    (fp_text value "Cathode" (at -0.762 -2.794) (layer "F.Fab")
-      (effects (font (size 1 1) (thickness 0.15)))
+    (fp_text value "Cathode" (at -0.254 -2.54) (layer "F.Fab")
+      (effects (font (size 0.75 0.75) (thickness 0.1)))
     )
     (fp_text user "${REFERENCE}" (at 0.7 2.5) (layer "F.Fab") hide
@@
   )
   (footprint "Package_TO_SOT_SMD:SOT-23-5" (layer "F.Cu")
-    (at 156.21 75.002 90)
+    (at 156.464 74.93 90)
     (descr "SOT, 5 Pin (https://www.jedec.org/sites/default/files/docs/Mo-178c.PDF variant AA), generated with kicad-footprint-generator ipc_gullwing_generator.py")
     (tags "SOT TO_SOT_SMD")
@@
   )
   (footprint "Resistor_SMD:R_0805_2012Metric" (layer "F.Cu")
-    (at 131.572 70.612)
-    (descr "Resistor SMD 0805 (2012 Metric), square (rectangular) end terminal, IPC_7351 nominal, (Body size source: IPC-SM-782 page 72, https://www.pcb-3d.com/wordpress/wp-content/uploads/ipc-sm-782a_amendment_1_and_2.pdf), generated with kicad-footprint-generator")
-    (tags "resistor")
+    (at 130.81 71.12)
+    (descr "Resistor SMD 0805 (2012 Metric), square (rectangular) end terminal, IPC_7351 nominal, (Body size source: IPC-SM-782 page 72, https://www.pcb-3d.com/wordpress/wp-content/uploads/ipc-sm-782a_amendment_1_and_2.pdf), generated with kicad-footprint-generator")
+    (tags "resistor")
