File: Kicad files/OpenHVPS-2/OpenHVPS-backups/OpenHVPS-2021-01-12_185036/OpenHVPS-2.kicad_sch (KiCad schematic)
At the start: 69 parts, among them J1 Conn_01x03_Male, J2 Conn_01x03_Male, Q1 FQT7N10, Q2 BC846, Q3 MMDT3906, U1 MAX6008AEUR+T, U2 74HC14, U3 MAX4162, U4 CD14538BM

Commit message: Updated all files
Parts:
- removed H1: Cathode, TestPoint:TestPoint_Loop_D3.80mm_Drill2.0mm, symbol Mechanical:MountingHole_Pad
- removed H2: Anode, TestPoint:TestPoint_Loop_D3.80mm_Drill2.0mm, symbol Mechanical:MountingHole_Pad
- removed J1: Conn_01x03_Male, Connector_PinHeader_2.54mm:PinHeader_1x03_P2.54mm_Vertical, symbol Connector:Conn_01x03_Male
- removed JP1: SolderJumper_2_Open, Jumper:SolderJumper-2_P1.3mm_Open_RoundedPad1.0x1.5mm, symbol Jumper:SolderJumper_2_Open
- removed R2: 10M, Resistor_SMD:R_1206_3216Metric, symbol Device:R
- R7: renamed from R1; value 10M -> 4M7
- renumbered C6 to C1, C17 to C10, C18 to C11, C20 to C12, C21 to C13, C1 to C14, C2 to C15, C3 to C16, C4 to C17, C5 to C18, C10 to C19, C7 to C2, C15 to C20, C19 to C21, C8 to C3, C9 to C4, C11 to C5, C12 to C6, C13 to C7, C14 to C8, C16 to C9, D3 to D1, D4 to D2, D5 to D3, D6 to D4, D7 to D5, D8 to D6, D9 to D7, D1 to D8, D2 to D9, FB2 to FB1, FB1 to FB2, J2 to J1, R10 to R1, R5 to R10, R6 to R11, R11 to R12, R12 to R13, R13 to R14, R14 to R15, R15 to R16, R16 to R17, R17 to R18, R18 to R19, R9 to R2, R19 to R20, R8 to R3, R7 to R4, R23 to R5, R20 to R6, R3 to R8, R4 to R9, U2 to U1, U3 to U2, U4 to U3, U1 to U4
Connections:
- net GND: now also J1.3 (Pin_3); no longer J1.2 (Pin_2)
- net at D9.2 (A), U3.6 (Q): now also J1.2 (Pin_2); no longer J1.3 (Pin_3)
Other:
- title: SafePulse -> OpenRover
- moved on the sheet: C1, C10, C11, C12, C13, C14, C15, C16, C17, C18, C19, C2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
