File: Kicad files/OpenHVPS-4/OpenRover-4.kicad_sch (KiCad schematic)
At the start: 69 parts, among them J1 Conn_01x03_Male, J2 Conn_01x03_Male, Q1 FQT7N10, Q2 BC846A, Q3 MMDT3906, U1 MAX6008AEUR+T, U2 74HC14, U3 MAX4162, U4 CD14538BM

Commit message: Update C22
Parts:
- C22: value 1nF -> 360pF
Other:
- moved on the sheet: R22
Changed lines of the file:
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@@
   (junction (at 252.73 133.985) (diameter 1.016) (color 0 0 0 0))
   (junction (at 254 99.695) (diameter 1.016) (color 0 0 0 0))
-  (junction (at 261.62 133.985) (diameter 1.016) (color 0 0 0 0))
-  (junction (at 261.62 150.495) (diameter 1.016) (color 0 0 0 0))
+  (junction (at 263.525 133.985) (diameter 1.016) (color 0 0 0 0))
+  (junction (at 263.525 150.495) (diameter 1.016) (color 0 0 0 0))
   (junction (at 275.59 99.695) (diameter 1.016) (color 0 0 0 0))
   (wire (pts (xy 22.86 97.155) (xy 30.48 97.155))
@@
     (stroke (width 0) (type solid) (color 0 0 0 0))
   )
-  (wire (pts (xy 252.73 133.985) (xy 261.62 133.985))
+  (wire (pts (xy 252.73 133.985) (xy 263.525 133.985))
     (stroke (width 0) (type solid) (color 0 0 0 0))
   )
@@
     (stroke (width 0) (type solid) (color 0 0 0 0))
   )
-  (wire (pts (xy 252.73 150.495) (xy 261.62 150.495))
+  (wire (pts (xy 252.73 150.495) (xy 263.525 150.495))
     (stroke (width 0) (type solid) (color 0 0 0 0))
   )
@@
     (stroke (width 0) (type solid) (color 0 0 0 0))
   )
-  (wire (pts (xy 261.62 133.985) (xy 261.62 140.335))
-    (stroke (width 0) (type solid) (color 0 0 0 0))
-  )
-  (wire (pts (xy 261.62 133.985) (xy 266.7 133.985))
-    (stroke (width 0) (type solid) (color 0 0 0 0))
-  )
-  (wire (pts (xy 261.62 147.955) (xy 261.62 150.495))
-    (stroke (width 0) (type solid) (color 0 0 0 0))
-  )
-  (wire (pts (xy 261.62 150.495) (xy 261.62 154.305))
+  (wire (pts (xy 263.525 133.985) (xy 263.525 140.335))
+    (stroke (width 0) (type solid) (color 0 0 0 0))
+  )
+  (wire (pts (xy 263.525 133.985) (xy 266.7 133.985))
+    (stroke (width 0) (type solid) (color 0 0 0 0))
+  )
+  (wire (pts (xy 263.525 147.955) (xy 263.525 150.495))
+    (stroke (width 0) (type solid) (color 0 0 0 0))
+  )
+  (wire (pts (xy 263.525 150.495) (xy 263.525 154.305))
     (stroke (width 0) (type solid) (color 0 0 0 0))
   )
@@
     )
   )
-  (symbol (lib_id "power:GND") (at 261.62 154.305 0) (unit 1)
-    (in_bom yes) (on_board yes)
-    (property "Reference" "#PWR025" (id 0) (at 261.62 160.655 0)
-      (effects (font (size 1.27 1.27)) hide)
-    )
-    (property "Value" "GND" (id 1) (at 261.7343 158.6294 0))
-    (property "Footprint" "" (id 2) (at 261.62 154.305 0)
-      (effects (font (size 1.27 1.27)) hide)
-    )
-    (property "Datasheet" "" (id 3) (at 261.62 154.305 0)
+  (symbol (lib_id "power:GND") (at 263.525 154.305 0) (unit 1)
+    (in_bom yes) (on_board yes)
+    (property "Reference" "#PWR025" (id 0) (at 263.525 160.655 0)
+      (effects (font (size 1.27 1.27)) hide)
+    )
+    (property "Value" "GND" (id 1) (at 263.6393 158.6294 0))
+    (property "Footprint" "" (id 2) (at 263.525 154.305 0)
+      (effects (font (size 1.27 1.27)) hide)
+    )
+    (property "Datasheet" "" (id 3) (at 263.525 154.305 0)
       (effects (font (size 1.27 1.27)) hide)
     )
@@
     )
   )
-  (symbol (lib_id "Device:R") (at 261.62 144.145 0) (unit 1)
-    (in_bom yes) (on_board yes)
-    (property "Reference" "R22" (id 0) (at 263.3981 142.9956 0)
-      (effects (font (size 1.27 1.27)) (justify left))
-    )
-    (property "Value" "20k" (id 1) (at 263.398 145.294 0)
-      (effects (font (size 1.27 1.27)) (justify left))
-    )
-    (property "Footprint" "Resistor_SMD:R_0805_2012Metric" (id 2) (at 259.842 144.145 90)
-      (effects (font (size 1.27 1.27)) hide)
-    )
-    (property "Datasheet" "https://www.digikey.com/en/products/detail/panasonic-electronic-components/ERJ-6ENF2002V/111532" (id 3) (at 261.62 144.145 0)
+  (symbol (lib_id "Device:R") (at 263.525 144.145 0) (unit 1)
+    (in_bom yes) (on_board yes)
+    (property "Reference" "R22" (id 0) (at 265.3031 142.9956 0)
+      (effects (font (size 1.27 1.27)) (justify left))
+    )
+    (property "Value" "20k" (id 1) (at 265.303 145.294 0)
+      (effects (font (size 1.27 1.27)) (justify left))
+    )
+    (property "Footprint" "Resistor_SMD:R_0805_2012Metric" (id 2) (at 261.747 144.145 90)
+      (effects (font (size 1.27 1.27)) hide)
+    )
+    (property "Datasheet" "https://www.digikey.com/en/products/detail/panasonic-electronic-components/ERJ-6ENF2002V/111532" (id 3) (at 263.525 144.145 0)
       (effects (font (size 1.27 1.27)) hide)
     )
@@
       (effects (font (size 1.27 1.27)) (justify left))
     )
-    (property "Value" "1nF" (id 1) (at 255.651 145.294 0)
+    (property "Value" "360pF" (id 1) (at 255.651 145.294 0)
       (effects (font (size 1.27 1.27)) (justify left))
     )
@@
     )
     (path "/743b7e51-503f-44bc-a063-83e91538f340"
-      (reference "C22") (unit 1) (value "1nF") (footprint "Capacitor_SMD:C_0805_2012Metric")
+      (reference "C22") (unit 1) (value "360pF") (footprint "Capacitor_SMD:C_0805_2012Metric")
     )
     (path "/00000000-0000-0000-0000-0000600ddc6a"
