File: Kicad files/OpenHVPS-5/Simulation/test simulation/test simulation.kicad_sch (KiCad schematic)
At the start: 9 parts, among them U1 MAX4162

Commit message: Updated V1.2.0
Parts:
- added L1: 4.7u, symbol pspice:INDUCTOR
- added M1: MNMOS, symbol pspice:MNMOS
Connections:
- net GND: now also M1.3 (S)
- net VDD: now also L1.2
- net Vout: now also M1.2 (G)
- new net MOSFET out: L1.1, M1.1 (D)
Other:
- note added: ".ac dec 66 1Hz 1kHz"
- note removed: ".ac dec 10 1 1Meg"
Changed lines of the file:
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@@
   (junction (at 219.075 111.76) (diameter 1.016) (color 0 0 0 0))
   (junction (at 238.76 53.34) (diameter 1.016) (color 0 0 0 0))
+  (junction (at 239.395 103.505) (diameter 1.016) (color 0 0 0 0))
   (junction (at 245.11 40.64) (diameter 1.016) (color 0 0 0 0))
   (junction (at 245.11 53.34) (diameter 1.016) (color 0 0 0 0))
@@
     (stroke (width 0) (type solid) (color 0 0 0 0))
   )
-  (wire (pts (xy 219.075 111.76) (xy 226.06 111.76))
+  (wire (pts (xy 219.075 111.76) (xy 231.775 111.76))
     (stroke (width 0) (type solid) (color 0 0 0 0))
   )
@@
     (stroke (width 0) (type solid) (color 0 0 0 0))
   )
+  (wire (pts (xy 239.395 101.6) (xy 239.395 103.505))
+    (stroke (width 0) (type solid) (color 0 0 0 0))
+  )
+  (wire (pts (xy 239.395 103.505) (xy 239.395 106.68))
+    (stroke (width 0) (type solid) (color 0 0 0 0))
+  )
+  (wire (pts (xy 239.395 103.505) (xy 255.905 103.505))
+    (stroke (width 0) (type solid) (color 0 0 0 0))
+  )
+  (wire (pts (xy 239.395 116.84) (xy 239.395 121.285))
+    (stroke (width 0) (type solid) (color 0 0 0 0))
+  )
   (wire (pts (xy 245.11 40.64) (xy 245.11 41.91))
     (stroke (width 0) (type solid) (color 0 0 0 0))
@@
     (stroke (width 0) (type solid) (color 0 0 0 0))
   )
-  (text ".ac dec 10 1 1Meg\n" (at 201.295 139.065 0)
+  (text "\n.ac dec 66 1Hz 1kHz \n" (at 227.33 138.43 180)
+    (effects (font (size 1.524 1.524)) (justify right bottom))
+  )
+  (label "Vout" (at 217.17 111.76 0)
     (effects (font (size 1.524 1.524)) (justify left bottom))
   )
-  (label "Vout" (at 217.17 111.76 0)
+  (label "MOSFET out" (at 255.905 103.505 0)
     (effects (font (size 1.524 1.524)) (justify left bottom))
   )
@@
     (pin "1")
   )
+  (symbol (lib_id "sallen_key_schlib:VDD") (at 239.395 88.9 0) (unit 1)
+    (in_bom yes) (on_board yes)
+    (property "Reference" "#PWR04" (id 0) (at 239.395 92.71 0)
+      (effects (font (size 1.27 1.27)) hide)
+    )
+    (property "Value" "VDD" (id 1) (at 239.8268 84.5058 0))
+    (property "Footprint" "" (id 2) (at 239.395 88.9 0))
+    (property "Datasheet" "" (id 3) (at 239.395 88.9 0))
+    (pin "1")
+  )
   (symbol (lib_id "sallen_key_schlib:VDD") (at 245.11 40.64 0) (unit 1)
     (in_bom yes) (on_board yes)
@@
     (property "Footprint" "" (id 2) (at 238.76 54.61 0))
     (property "Datasheet" "" (id 3) (at 238.76 54.61 0))
+    (pin "1")
+  )
+  (symbol (lib_id "power:GND") (at 239.395 121.285 0) (unit 1)
+    (in_bom yes) (on_board yes)
+    (property "Reference" "#PWR08" (id 0) (at 239.395 127.635 0)
+      (effects (font (size 1.27 1.27)) hide)
+    )
+    (property "Value" "GND" (id 1) (at 239.522 125.6792 0))
+    (property "Footprint" "" (id 2) (at 239.395 121.285 0)
+      (effects (font (size 1.27 1.27)) hide)
+    )
+    (property "Datasheet" "" (id 3) (at 239.395 121.285 0)
+      (effects (font (size 1.27 1.27)) hide)
+    )
     (pin "1")
   )
@@
     (pin "2")
   )
+  (symbol (lib_id "pspice:INDUCTOR") (at 239.395 95.25 90) (unit 1)
+    (in_bom yes) (on_board yes)
+    (property "Reference" "L1" (id 0) (at 240.4111 94.4891 90)
+      (effects (font (size 1.27 1.27)) (justify right))
+    )
+    (property "Value" "4.7u" (id 1) (at 240.4111 96.7878 90)
+      (effects (font (size 1.27 1.27)) (justify right))
+    )
+    (property "Footprint" "" (id 2) (at 239.395 95.25 0)
+      (effects (font (size 1.27 1.27)) hide)
+    )
+    (property "Datasheet" "~" (id 3) (at 239.395 95.25 0)
+      (effects (font (size 1.27 1.27)) hide)
+    )
+    (pin "1")
+    (pin "2")
+  )
   (symbol (lib_id "sallen_key_schlib:C") (at 177.8 119.38 0) (unit 1)
     (in_bom yes) (on_board yes)
@@
     (pin "2")
   )
+  (symbol (lib_id "pspice:MNMOS") (at 236.855 111.76 0) (unit 1)
+    (in_bom yes) (on_board yes)
+    (property "Reference" "M1" (id 0) (at 242.9511 110.9991 0)
+      (effects (font (size 1.27 1.27)) (justify left))
+    )
+    (property "Value" "MNMOS" (id 1) (at 242.9511 113.2978 0)
+      (effects (font (size 1.27 1.27)) (justify left))
+    )
+    (property "Footprint" "" (id 2) (at 236.22 111.76 0)
+      (effects (font (size 1.27 1.27)) hide)
+    )
+    (property "Datasheet" "~" (id 3) (at 236.22 111.76 0)
+      (effects (font (size 1.27 1.27)) hide)
+    )
+    (property "Spice_Primitive" "I" (id 4) (at 236.855 111.76 0)
+      (effects (font (size 1.27 1.27)) hide)
+    )
+    (property "Spice_Netlist_Enabled" "Y" (id 5) (at 236.855 111.76 0)
+      (effects (font (size 1.27 1.27)) hide)
+    )
+    (pin "1")
+    (pin "2")
+    (pin "3")
+    (pin "4")
+  )
   (symbol (lib_id "sallen_key_schlib:Generic_Opamp") (at 199.39 111.76 0) (unit 1)
     (in_bom yes) (on_board yes)
@@
       (reference "#PWR03") (unit 1) (value "VDD") (footprint "")
     )
+    (path "/add57f0b-9b65-4609-88ef-d92479f08ca4"
+      (reference "#PWR04") (unit 1) (value "VDD") (footprint "")
+    )
     (path "/00000000-0000-0000-0000-0000578902d2"
       (reference "#PWR05") (unit 1) (value "GND") (footprint "")
@@
       (reference "#PWR07") (unit 1) (value "VSS") (footprint "")
     )
+    (path "/458bad65-71c1-408a-8155-1be630bd4372"
+      (reference "#PWR08") (unit 1) (value "GND") (footprint "")
+    )
     (path "/00000000-0000-0000-0000-00005a0b57f1"
       (reference "#PWR0101") (unit 1) (value "GND") (footprint "")
@@
       (reference "C2") (unit 1) (value "100pF") (footprint "Capacitor_SMD:C_0805_2012Metric")
     )
+    (path "/98b3f8e9-46fb-4c69-a4d3-7297116116b4"
+      (reference "L1") (unit 1) (value "4.7u") (footprint "")
+    )
+    (path "/cde6f2c9-55db-4317-a8b3-6b5652059c3b"
+      (reference "M1") (unit 1) (value "MNMOS") (footprint "")
+    )
     (path "/d69240ad-8b6d-473a-bd72-401d009649a6"
