File: Kicad files/OpenHVPS-5/OpenHVPS-5.kicad_sch (KiCad schematic)
At the start: 87 parts, among them J1 Conn_01x03_Male, Q1 FQT7N10L, Q2 BC846A, Q3 MMBT3906, Q4 MMBT3906, U1 MAX6006AEUR+T, U2 74HC14, U3 MAX4162, U4 CD14538BM

Commit message: Updated V1.2.0
Parts:
- removed C26: 100pF, Capacitor_SMD:C_0805_2012Metric, symbol Device:C
- C1: Digikey (none) -> 732-12190-1-ND
- C10, C11, C12, C13, C14, C15, C16, C17, C18, C6, C7, C8, C9: Digikey (none) -> 445-6808-1-ND
- C19, C2, C23, C27, C5: Digikey (none) -> 1276-6455-1-ND
- C22: Digikey (none) -> 1276-1303-1-ND
- C24: Digikey (none) -> 1276-1015-1-ND
- C25: value 1nF -> 10nF; Digikey (none) -> 1276-1015-1-ND
- C3: Digikey (none) -> 478-1371-1-ND
- C4: Digikey (none) -> 587-5425-1-ND
- D1, D2: Digikey (none) -> 1727-4797-1-ND
- D3, D4, D5, D6, D7, D8, D9: Digikey (none) -> BAV23SFSCT-ND
- F1: Digikey (none) -> 490-8510-1-ND
- FB1, FB2: value BKP2125HS221-T -> 74279220321; Digikey (none) -> 732-6125-1-ND
- L1: Digikey (none) -> 587-4451-1-ND
- Q1: Digikey (none) -> FQT7N10LTFCT-ND
- Q2: Digikey (none) -> BC846A-7FDICT-ND
- Q3, Q4: Digikey (none) -> MMBT3906LT1GOSCT-ND
- R1: Digikey (none) -> RHM4.7MAICT-ND
- R10, R7, R8, R9: Digikey (none) -> RMCF0805FT22M0CT-ND
- R11: Digikey (none) -> A129767CT-ND
- R12, R25: Digikey (none) -> A106053CT-ND
- R13, R19, R3: Digikey (none) -> RMCF0805FT100KCT-ND
- R15: Digikey (none) -> 311-392KCRCT-ND
- R16: Digikey (none) -> YAG3361CT-ND
- R17: Digikey (none) -> RMCF0805FT499KCT-ND
- R18: Digikey (none) -> RNCP0805FTD1K00CT-ND
- R20: value 330K -> 118K; Digikey A126361CT-ND -> 311-118KCRCT-ND
- R21: Digikey (none) -> 311-47.0KCRCT-ND
- R22: Digikey (none) -> RMCF0805FT20K0CT-ND
- R24: value 22M -> 33k; Digikey (none) -> A129767CT-ND
- R26: Digikey (none) -> 408-1556-1-ND
- R4: Digikey (none) -> RNCP0805FTD10K0CT-ND
- R6: Digikey (none) -> 2019-RK73H2ATTD1213FCT-ND
- U1: value MAX6006AEUR+T -> TS4061AILT-1.25; Digikey MAX6006AEUR+TCT-ND -> 497-15222-1-ND
- U2: Digikey (none) -> 296-9179-1-ND
- U3: value MAX4162 -> TLV27L1IDBVT; Digikey (none) -> 296-26814-1-ND
- U4: Digikey (none) -> 296-32849-5-ND
Connections:
- net GND: now also R24.2; no longer R23.2
- net at R23.1, R7.1, U3.4 (-): no longer R24.2
- net at R24.1: now also R23.2
Other:
- moved on the sheet: R24

Commit message: Safepulse V1.2.1
Parts:
- added U33: MAX9910EXK+T, Package_TO_SOT_SMD:SOT-353_SC-70-5, symbol Amplifier_Operational:MCP6L01Ux-xOT
Connections:
- net GND: now also U33.2 (V-)
- net at R3.2, TP2.1, U3.1: now also U33.4
- net at R27.2, U3.3 (+): now also U33.1 (+)
- net at R23.1, R7.1, U3.4 (-): now also U33.3 (-)
- net at C27.1, R20.1, R25.2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: now also U33.5 (V+)
Other:
- moved on the sheet: C25, R23, R24, R27, R3, R7, R8, R9, TP1, TP2, U3

Commit message: Parts order for V1.2.1c
Parts:
- R1: Digikey10M (none) -> RHM10.0MAICT-ND
Changed lines of the file:
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@@
+      (effects (font (size 1.27 1.27)) hide)
+    )
+    (property "Digikey10M" "RHM10.0MAICT-ND" (id 5) (at 257.81 99.695 90)
       (effects (font (size 1.27 1.27)) hide)
     )
