File: Kicad files/Safepulse/SafePulse.kicad_sch (KiCad schematic)
At the start: 87 parts, among them J1 Conn_01x03_Male, Q1 FQT7N10L, Q2 BC846A, Q3 MMBT3906, Q4 MMBT3906, U1 TS4061AILT-1.25, U2 74HC14, U3 TLV27L1DBVT, U33 MAX9910EXK+T, U4 CD14538BM

Commit message: Merge branch 'main' of https://github.com/Safecast/open-hvps into main
Parts:
- added IC1: S-35770E01I-K8T2U, SOP65P400X80-8N, symbol S-35770E01I-K8T2U:S-35770E01I-K8T2U
- added J2: 4208, 4208, symbol 4208:4208
Connections:
- net +3V3: now also IC1.8 (VDD), J2.4
- net GND: now also IC1.4 (VSS), J2.1
- new net: IC1.6 (SDA), J2.2
- new net: IC1.7 (SCL), J2.3
Changed lines of the file:
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@@
-(kicad_sch (version 20210406) (generator eeschema)
+(kicad_sch (version 20210621) (generator eeschema)
   (paper "A4")
   (title_block
@@
   (junction (at 115.57 99.695) (diameter 1.016) (color 0 0 0 0))
   (junction (at 115.57 145.415) (diameter 1.016) (color 0 0 0 0))
+  (junction (at 125.73 53.34) (diameter 1.016) (color 0 0 0 0))
   (junction (at 126.365 99.695) (diameter 1.016) (color 0 0 0 0))
   (junction (at 129.54 177.165) (diameter 1.016) (color 0 0 0 0))
   (junction (at 132.08 78.105) (diameter 1.016) (color 0 0 0 0))
   (junction (at 135.89 145.415) (diameter 1.016) (color 0 0 0 0))
+  (junction (at 142.875 53.34) (diameter 1.016) (color 0 0 0 0))
   (junction (at 143.51 99.695) (diameter 1.016) (color 0 0 0 0))
   (junction (at 143.51 108.585) (diameter 1.016) (color 0 0 0 0))
@@
   (junction (at 170.18 78.105) (diameter 1.016) (color 0 0 0 0))
   (junction (at 170.18 88.265) (diameter 1.016) (color 0 0 0 0))
+  (junction (at 173.355 38.735) (diameter 1.016) (color 0 0 0 0))
   (junction (at 176.53 126.365) (diameter 1.016) (color 0 0 0 0))
   (junction (at 179.07 99.695) (diameter 1.016) (color 0 0 0 0))
@@
     (stroke (width 0) (type solid) (color 0 0 0 0))
   )
+  (wire (pts (xy 115.57 20.955) (xy 173.355 20.955))
+    (stroke (width 0) (type solid) (color 0 0 0 0))
+  )
   (wire (pts (xy 115.57 26.035) (xy 115.57 20.955))
     (stroke (width 0) (type solid) (color 0 0 0 0))
@@
     (stroke (width 0) (type solid) (color 0 0 0 0))
   )
-  (wire (pts (xy 125.73 55.245) (xy 125.73 51.435))
+  (wire (pts (xy 125.73 53.34) (xy 125.73 51.435))
+    (stroke (width 0) (type solid) (color 0 0 0 0))
+  )
+  (wire (pts (xy 125.73 55.245) (xy 125.73 53.34))
     (stroke (width 0) (type solid) (color 0 0 0 0))
   )
@@
     (stroke (width 0) (type solid) (color 0 0 0 0))
   )
+  (wire (pts (xy 142.875 46.355) (xy 142.875 53.34))
+    (stroke (width 0) (type solid) (color 0 0 0 0))
+  )
+  (wire (pts (xy 142.875 53.34) (xy 125.73 53.34))
+    (stroke (width 0) (type solid) (color 0 0 0 0))
+  )
   (wire (pts (xy 143.51 93.345) (xy 143.51 99.695))
     (stroke (width 0) (type solid) (color 0 0 0 0))
@@
     (stroke (width 0) (type solid) (color 0 0 0 0))
   )
+  (wire (pts (xy 173.355 38.735) (xy 173.355 20.955))
+    (stroke (width 0) (type solid) (color 0 0 0 0))
+  )
+  (wire (pts (xy 173.355 38.735) (xy 181.61 38.735))
+    (stroke (width 0) (type solid) (color 0 0 0 0))
+  )
+  (wire (pts (xy 173.355 41.275) (xy 181.61 41.275))
+    (stroke (width 0) (type solid) (color 0 0 0 0))
+  )
+  (wire (pts (xy 173.355 43.815) (xy 181.61 43.815))
+    (stroke (width 0) (type solid) (color 0 0 0 0))
+  )
   (wire (pts (xy 173.99 99.695) (xy 179.07 99.695))
     (stroke (width 0) (type solid) (color 0 0 0 0))
@@
     (stroke (width 0) (type solid) (color 0 0 0 0))
   )
+  (wire (pts (xy 181.61 46.355) (xy 181.61 53.34))
+    (stroke (width 0) (type solid) (color 0 0 0 0))
+  )
+  (wire (pts (xy 181.61 53.34) (xy 142.875 53.34))
+    (stroke (width 0) (type solid) (color 0 0 0 0))
+  )
   (wire (pts (xy 181.61 78.105) (xy 187.96 78.105))
     (stroke (width 0) (type solid) (color 0 0 0 0))
@@
     (pin "4")
   )
+  (symbol (lib_id "4208:4208") (at 201.93 46.355 180) (unit 1)
+    (in_bom yes) (on_board yes) (fields_autoplaced)
+    (property "Reference" "J2" (id 0) (at 191.77 32.2792 0))
+    (property "Value" "4208" (id 1) (at 191.77 35.0543 0))
+    (property "Footprint" "4208" (id 2) (at 185.42 48.895 0)
+      (effects (font (size 1.27 1.27)) (justify left) hide)
+    )
+    (property "Datasheet" "https://cdn-shop.adafruit.com/product-files/4208/4208_Kaweei_C13396_diagram.pdf" (id 3) (at 185.42 46.355 0)
+      (effects (font (size 1.27 1.27)) (justify left) hide)
+    )
+    (property "Description" "Adafruit Accessories JST SH 4-pin Right Angle Connector (10-pack) - Qwiic Compatible" (id 4) (at 185.42 43.815 0)
+      (effects (font (size 1.27 1.27)) (justify left) hide)
+    )
+    (property "Height" "3.05" (id 5) (at 185.42 41.275 0)
+      (effects (font (size 1.27 1.27)) (justify left) hide)
+    )
+    (property "Manufacturer_Name" "Adafruit" (id 6) (at 185.42 38.735 0)
+      (effects (font (size 1.27 1.27)) (justify left) hide)
+    )
+    (property "Manufacturer_Part_Number" "4208" (id 7) (at 185.42 36.195 0)
+      (effects (font (size 1.27 1.27)) (justify left) hide)
+    )
+    (property "Mouser Part Number" "485-4208" (id 8) (at 185.42 33.655 0)
+      (effects (font (size 1.27 1.27)) (justify left) hide)
+    )
+    (property "Mouser Price/Stock" "https://www.mouser.co.uk/ProductDetail/Adafruit/4208?qs=PzGy0jfpSMtbScLbr0L5dw%3D%3D" (id 9) (at 185.42 31.115 0)
+      (effects (font (size 1.27 1.27)) (justify left) hide)
+    )
+    (property "Arrow Part Number" "" (id 10) (at 185.42 28.575 0)
+      (effects (font (size 1.27 1.27)) (justify left) hide)
+    )
+    (property "Arrow Price/Stock" "" (id 11) (at 185.42 26.035 0)
+      (effects (font (size 1.27 1.27)) (justify left) hide)
+    )
+    (pin "1")
+    (pin "2")
+    (pin "3")
+    (pin "4")
+    (pin "5")
+    (pin "6")
+  )
   (symbol (lib_id "74xx:74HC14") (at 24.13 50.165 0) (unit 7)
     (in_bom yes) (on_board yes)
@@
     (pin "8")
   )
+  (symbol (lib_id "S-35770E01I-K8T2U:S-35770E01I-K8T2U") (at 142.875 38.735 0) (unit 1)
+    (in_bom yes) (on_board yes) (fields_autoplaced)
+    (property "Reference" "IC1" (id 0) (at 158.115 32.2792 0))
+    (property "Value" "S-35770E01I-K8T2U" (id 1) (at 158.115 35.0543 0))
+    (property "Footprint" "SOP65P400X80-8N" (id 2) (at 169.545 36.195 0)
+      (effects (font (size 1.27 1.27)) (justify left) hide)
+    )
+    (property "Datasheet" "https://www.mouser.com/datasheet/2/360/S35770_I_E-1628617.pdf" (id 3) (at 169.545 38.735 0)
+      (effects (font (size 1.27 1.27)) (justify left) hide)
+    )
+    (property "Description" "Timers & Support Products Counter IC with 2-wire(I2C-bus) interface" (id 4) (at 169.545 41.275 0)
+      (effects (font (size 1.27 1.27)) (justify left) hide)
+    )
+    (property "Height" "0.8" (id 5) (at 169.545 43.815 0)
+      (effects (font (size 1.27 1.27)) (justify left) hide)
+    )
+    (property "Manufacturer_Name" "ABLIC U.S.A. Inc." (id 6) (at 169.545 46.355 0)
+      (effects (font (size 1.27 1.27)) (justify left) hide)
+    )
+    (property "Manufacturer_Part_Number" "S-35770E01I-K8T2U" (id 7) (at 169.545 48.895 0)
+      (effects (font (size 1.27 1.27)) (justify left) hide)
+    )
+    (property "Mouser Part Number" "628-S35770E01I-K8T2U" (id 8) (at 169.545 51.435 0)
+      (effects (font (size 1.27 1.27)) (justify left) hide)
+    )
+    (property "Mouser Price/Stock" "https://www.mouser.co.uk/ProductDetail/ABLIC/S-35770E01I-K8T2U?qs=vLWxofP3U2yvSXNQEw14rA%3D%3D" (id 9) (at 169.545 53.975 0)
+      (effects (font (size 1.27 1.27)) (justify left) hide)
+    )
+    (property "Arrow Part Number" "" (id 10) (at 169.545 56.515 0)
+      (effects (font (size 1.27 1.27)) (justify left) hide)
+    )
+    (property "Arrow Price/Stock" "" (id 11) (at 169.545 59.055 0)
+      (effects (font (size 1.27 1.27)) (justify left) hide)
+    )
+    (pin "1")
+    (pin "2")
+    (pin "3")
+    (pin "4")
+    (pin "5")
+    (pin "6")
+    (pin "7")
+    (pin "8")
+  )
   (symbol (lib_id "4xxx:4538") (at 83.82 161.925 0) (unit 2)
     (in_bom yes) (on_board yes)
@@
       (reference "H4") (unit 1) (value "Anode") (footprint "TestPoint:TestPoint_Loop_D3.50mm_Drill1.4mm_Beaded")
     )
+    (path "/a90c6a18-b5af-43af-a9f1-c016c49a81d8"
+      (reference "IC1") (unit 1) (value "S-35770E01I-K8T2U") (footprint "SOP65P400X80-8N")
+    )
     (path "/cfef5cd8-f134-487a-8cb2-e8668492f6e4"
       (reference "J1") (unit 1) (value "Conn_01x03_Male") (footprint "Connector_PinHeader_2.54mm:PinHeader_1x03_P2.54mm_Vertical")
     )
+    (path "/0aa6faca-6bcf-4123-bf4f-61c6365d2bac"
+      (reference "J2") (unit 1) (value "4208") (footprint "4208")
+    )
     (path "/00000000-0000-0000-0000-00005ffe44be"
