File: Kicad files/Safepulse/SafePulse.kicad_pcb (KiCad board)
At the start: 4 copper layers, 40.6 x 20.8 mm, 89 parts, among them IC1 S-35770E01I-K8T2U, J1 Conn_01x03_Male, J2 4208, Q1 FQT7N10L, Q2 BC846A, Q3 MMBT3906, Q4 MMBT3906, U1 TS4061AILT-1.25, U2 74HC14, U3 TLV27L1DBVT, U33 MAX9910EXK+T, U4 CD14538BM

Commit message: V1.2.3 (allan)
Parts:
- removed R26: 0.1E, Resistor_SMD:R_0805_2012Metric
- removed TP10: TestPoint, TestPoint:TestPoint_Pad_1.0x1.0mm
- C4: value 47uF -> 10uF; footprint Capacitor_SMD:C_1210_3225Metric -> Capacitor_SMD:C_0805_2012Metric
- IC1: moved to F.Cu
- moved J2 34.5 mm to (130.0, 70.0), turned to 90 degrees
- moved IC1 12.6 mm to (132.1, 71.6), turned to 180 degrees
- moved TP3 11.4 mm to (141.1, 62.8)
- moved C4 6.58 mm to (135.8, 74.0), turned to -90 degrees
- moved TP4 5.73 mm to (129.6, 62.4)
- moved TP5 4.60 mm to (129.6, 64.5)
- moved TP8 4.37 mm to (142.8, 76.8)
- moved F1 0.99 mm to (127.6, 71.9)
- moved U2 0.95 mm to (135.3, 61.8)
- moved R11 0.56 mm to (141.6, 75.2)
- moved C2 0.46 mm to (129.6, 59.6)
- moved D1 0.45 mm to (134.8, 67.9)
- moved R4 0.38 mm to (136.8, 68.0)
- moved R12 0.35 mm to (142.1, 72.7)
- moved R21 0.34 mm to (142.1, 74.8)
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Connections:
- C5 pad 1: Net-(D2-Pad2) -> Net-(C5-Pad1)
- FB2 pad 2: Net-(D2-Pad2) -> Net-(C5-Pad1)
- L1 pad 1: Net-(D2-Pad2) -> Net-(C5-Pad1)
- Q1 pad 3: Net-(Q1-Pad3) -> GND
Routing:
- net GND: track 112.2 -> 64.3 mm
- net Net-(C5-Pad1): track 0.00 -> 6.90 mm
- net Net-(IC1-Pad7): track 0.00 -> 6.79 mm, vias 0 -> 2
- net Net-(D2-Pad2): track 50.0 -> 43.9 mm
- net Net-(Q1-Pad3): track 5.96 -> 0.00 mm, vias 1 -> 0
- net Net-(IC1-Pad6): track 0.00 -> 4.92 mm, vias 0 -> 1
- net Net-(C7-Pad1): track 18.4 -> 23.0 mm
- net Net-(R6-Pad1): track 22.0 -> 23.3 mm, vias 0 -> 2
- net +3V3: track 38.2 -> 37.0 mm, vias 3 -> 4
- net Net-(Q1-Pad1): track 28.6 -> 27.5 mm, vias 1 -> 2
- net Net-(D1-Pad1): track 27.2 -> 28.1 mm
- net Net-(F1-Pad1): track 3.15 -> 3.82 mm
- net (no net): vias 2 -> 0

Commit message: Fixed QR logo
Parts:
- added REF**: LOGO, Library:QR_code_SafePulse, F.Cu at (156.2, 63.6)
