File: SafePulse.kicad_sch (KiCad schematic)
At the start: 87 parts, among them IC1 S-35770E01I-K8T2U, J1 Conn_01x03_Male, J2 4208, Q1 FQT7N10L, Q2 BC846A, Q3 MMBT3906, Q4 MMBT3906, U1 TS4061AICT-1.25, U2 74HC14, U3 TLV27L1DBVT, U33 MAX9910EXK+T, U4 CD14538BM

Commit message: added Allan changes
Parts:
- C1: LCSC (none) -> C520084
- C10, C11, C12, C13, C14, C15, C16, C17, C18, C6, C7, C8, C9: LCSC (none) -> C710458
- C19, C2, C23, C27, C4, C5: LCSC (none) -> C1713
- C22: LCSC (none) -> C1717
- C24: LCSC (none) -> C97905
- C25: LCSC (none) -> C19110
- C3: LCSC (none) -> C83170
- D1, D2: LCSC (none) -> C282360
- D3, D4, D5, D6, D7, D8, D9: LCSC (none) -> C151049
- F1: LCSC (none) -> C20978
- FB1, FB2: LCSC (none) -> C515370
- L1: LCSC (none) -> C359308
- Q1: LCSC (none) -> C154506
- Q2: LCSC (none) -> C507907
- Q3, Q4: LCSC (none) -> C53444
- R1: LCSC (none) -> C488845
- R10, R7, R8, R9: LCSC (none) -> C34719
- R11: LCSC (none) -> C242487
- R12, R25, R5: LCSC (none) -> C328380
- R13, R19, R3: LCSC (none) -> C96346
- R14: LCSC (none) -> C865422
- R15: LCSC (none) -> C104108
- R16: LCSC (none) -> C107700
- R17: LCSC (none) -> C317482
- R18: LCSC (none) -> C95781
- R20: LCSC (none) -> C228266
- R21: LCSC (none) -> C328397
- R22: LCSC (none) -> C17444
- R23, R27: LCSC (none) -> C422787
- R24: LCSC (none) -> C352242
- R4: LCSC (none) -> C161788
- R6: LCSC (none) -> C17438
- U1: LCSC (none) -> C5267733
- U2: LCSC (none) -> C232776
- U33: LCSC (none) -> C2057992
- U4: LCSC (none) -> C56163

Commit message: Updated BOM and position files for JLCPCB
Parts:
- R11: LCSC C242487 -> C1739
- R20: LCSC C228266 -> C101434
- R4: LCSC C161788 -> C17414
- U3: LCSC (none) -> C2868527
Changed lines of the file:
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@@
 			)
 		)
-		(property "LCSC" "C228266"
+		(property "LCSC" "C101434"
 			(at 42.418 108.687 0)
 			(effects
@@
 			)
 		)
-		(property "LCSC" "C161788"
+		(property "LCSC" "C17414"
 			(at 60.96 53.7972 0)
 			(effects
@@
 			)
 		)
-		(property "LCSC" "C242487"
+		(property "LCSC" "C1739"
 			(at 161.29 105.8672 0)
 			(effects
@@
 			(effects
 				(font
+					(size 1.27 1.27)
+				)
+				(hide yes)
+			)
+		)
+		(property "LCSC" "C2868527"
+			(at 52.07 160.6549 0)
+			(effects
+				(font

Commit message: Updated V1.2.4 board with new JCLPCB number
Parts:
- C1: LCSC C520084 -> C1716
Changed lines of the file:
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@@
 			)
 		)
-		(property "LCSC" "C520084"
+		(property "LCSC" "C1716"
 			(at 44.196 68.6816 0)
 			(effects

Commit message: V1.2.5 boards
Parts:
- C1: LCSC C1716 -> C520084
- Q2: footprint Package_TO_SOT_SMD:SOT-23 -> Package_TO_SOT_SMD:SOT-323_SC-70_Handsoldering
- U1: footprint Package_TO_SOT_SMD:SOT-323_SC-70 -> Package_TO_SOT_SMD:SOT-23
Changed lines of the file:
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@@
 			)
 		)
-		(property "Footprint" "Package_TO_SOT_SMD:SOT-323_SC-70"
+		(property "Footprint" "Package_TO_SOT_SMD:SOT-23"
 			(at 15.875 120.015 0)
 			(effects
@@
 			)
 		)
-		(property "LCSC" "C1716"
+		(property "LCSC" "C520084"
 			(at 44.196 68.6816 0)
 			(effects
@@
 			)
 		)
-		(property "Footprint" "Package_TO_SOT_SMD:SOT-23"
+		(property "Footprint" "Package_TO_SOT_SMD:SOT-323_SC-70_Handsoldering"
 			(at 190.5 137.16 0)
 			(effects

Commit message: Update layout for SOT-323 for U1 from a SOT-23 footprint
Parts:
- U1: footprint Package_TO_SOT_SMD:SOT-23 -> Package_TO_SOT_SMD:SOT-323_SC-70
Changed lines of the file:
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@@
 			)
 		)
-		(property "Footprint" "Package_TO_SOT_SMD:SOT-23"
+		(property "Footprint" "Package_TO_SOT_SMD:SOT-323_SC-70"
 			(at 15.875 120.015 0)
 			(effects

Commit message: V1.2.6 draft
Parts:
- J1: footprint Connector_PinHeader_2.54mm:PinHeader_1x03_P2.54mm_Vertical -> Connector_PinHeader_2.54mm:PinHeader_1x05_P2.54mm_Vertical; symbol Connector:Conn_01x03_Male -> Connector:Conn_01x05_Pin
Connections:
- net at IC1.6 (SDA), J2.3: now also J1.4 (Pin_4)
- net SDA: now reaches IC1.7 (SCL), J2.4
- net SDA: now also J1.5 (Pin_5)
Other:
- moved on the sheet: U1

Commit message: cleaned up files
Parts:
- removed U3: TLV27L1DBVT, Package_TO_SOT_SMD:SOT-23-5, symbol Amplifier_Operational:TLV2371DBV
- Q2: footprint Package_TO_SOT_SMD:SOT-323_SC-70_Handsoldering -> Package_TO_SOT_SMD:SOT-323_SC-70
Connections:
- net SDA: no longer IC1.7 (SCL), J1.5 (Pin_5), J2.4
- net at IC1.6 (SDA), J2.3: now also J1.5 (Pin_5); no longer J1.4 (Pin_4)
- new net: IC1.7 (SCL), J1.4 (Pin_4), J2.4
Other:
- moved on the sheet: IC1
