File: V200/SafePulse.kicad_pcb (KiCad board)
At the start: 4 copper layers, 40.6 x 20.8 mm, 91 parts, among them IC1 S-35770E01I-K8T2U, J1 Conn_01x03_Male, J2 JST SM04B-SRSS-TB(LF)(SN), Q1 FQT7N10L, Q2 BC846A, Q3 MMBT3906, Q4 MMBT3906, U1 TS4061AICT-1.25, U2 74HC14, U33 MAX9910EXK+T, U4 CD14538BM

Commit message: Updated with Allan new files
Parts:
- removed the G3 at (160.2, 65.7)
- removed the G3 at (163.9, 68.6)
- added G3: LOGO, Symbol:HV warning, F.Cu at (160.3, 65.6)
- added G3: LOGO, Symbol:HV warning, B.Cu at (163.7, 68.5)
- added R2: 10M, Resistor_SMD:R_1206_3216Metric, F.Cu at (165.4, 67.2)
- H2: value Anode -> LND712
- H4: value Anode -> LND7317
- moved R1 0.23 mm to (163.1, 67.2)
Connections:
- H4 pad 1: Net-(H2-Pad1) -> Net-(H4-Pad1)
- R1 pad 2: Net-(H2-Pad1) -> Net-(H4-Pad1)
Routing:
- net Net-(H4-Pad1): track 0.00 -> 8.12 mm
- net Net-(H2-Pad1): track 7.24 -> 3.61 mm
- net Net-(D9-A): track 11.7 -> 15.2 mm
Other:
- board text added: "Anode"
