File: V200/SafePulse.kicad_pcb (KiCad board)
At the start: 4 copper layers, 40.6 x 20.8 mm, 92 parts, among them IC1 S-35770E01I-K8T2U, J1 Conn_01x03_Male, J2 JST SM04B-SRSS-TB(LF)(SN), Q1 FQT7N10L, Q2 BC846A, Q3 MMBT3906, Q4 MMBT3906, U1 TS4061AICT-1.25, U2 74HC14, U33 MAX9910EXK+T, U4 CD14538BM

Commit message: V2.0.0 updated files
Parts:
- removed C20: 100pF, Capacitor_SMD:C_0805_2012Metric
- removed C21: 0.1uF, Capacitor_SMD:C_0805_2012Metric
- removed G3 (x2): LOGO, Symbol:HV warning
- removed R2: 10M, Resistor_SMD:R_1206_3216Metric
- removed R26: 22M, Resistor_SMD:R_0805_2012Metric
- C1: value 110pF -> 150pF
- C22: value 390pF -> 1.5nF
- C3: value 1nF -> 10nF
- C4: value 47uF -> 10uF
- H2: value LND712 -> Anode
- H4: value LND7317 -> Anode
- J2: value JST SM04B-SRSS-TB(LF)(SN) -> 4208
- R22: value 20K -> 12K
- R24: value 33k -> 22k
- TP7: moved to F.Cu
- moved R24 6.51 mm to (143.8, 58.3), turned to 180 degrees
- moved U33 2.17 mm to (145.0, 64.4), turned to -90 degrees
- moved R23 1.85 mm to (147.2, 58.3), turned to 180 degrees
- moved TP7 1.32 mm to (165.6, 65.9), turned to 0 degrees
- moved R27 0.72 mm to (148.1, 64.4)
- moved TP1 0.53 mm to (150.1, 66.0)
- moved TP2 0.48 mm to (144.5, 67.3)
- moved TP6 0.46 mm to (140.9, 58.3)
- moved C25 0.43 mm to (150.1, 63.3)
- moved R1 0.23 mm to (163.3, 67.2)
- moved TP9 0.09 mm to (147.8, 71.2)
Connections:
- C3 pad 2: Net-(U4A-VSS) -> GND
- H4 pad 1: Net-(H4-Pad1) -> Net-(H2-Pad1)
- IC1 pad 1: +3V3 -> unconnected-(IC1-~RST-Pad1)
- R1 pad 2: Net-(H4-Pad1) -> Net-(H2-Pad1)
- U4 pad 1: Net-(U4A-VSS) -> GND
- U4 pad 11: Net-(U4A-R) -> GND
- U4 pad 12: GND -> Net-(U4A-R)
- U4 pad 13: Net-(U4A-R) -> GND
- U4 pad 14: GND -> unconnected-(U4B-RxCx-Pad14)
- U4 pad 15: unconnected-(U4B-VSS-Pad15) -> GND
Routing:
- net Net-(H4-Pad1): track 8.12 -> 0.00 mm
- net Net-(U4A-VSS): track 7.41 -> 0.00 mm
- net GND: track 56.9 -> 51.2 mm, vias 7 -> 15
- net Net-(U4A-R): track 23.2 -> 18.0 mm
- net Net-(H2-Pad1): track 3.61 -> 7.24 mm
- net Net-(D9-A): track 15.2 -> 11.8 mm, vias 1 -> 0
- net Net-(IC1-SDA): track 17.0 -> 20.3 mm
- net Net-(U33-+): track 2.46 -> 5.26 mm
- net Net-(U33-V+): track 15.5 -> 13.1 mm
- net +3V3: track 41.2 -> 39.1 mm
- net Net-(R3-Pad2): track 9.28 -> 7.32 mm
- net Net-(C20-Pad1): track 1.70 -> 0.00 mm
- net Net-(C6-Pad2): track 13.8 -> 13.0 mm
- net Net-(D2-K): track 25.3 -> 25.8 mm
- net Net-(D2-A): track 44.0 -> 43.6 mm, vias 1 -> 0
Other:
- board text removed: "Anode"
- board text removed: "HIGH VOLTAGE 500V !!"
- board text removed: "SafePulse High Voltage Geiger Muller Power Supply Ver 2.0.0 01 Nov 2025"

Commit message: One more fix
Other:
- board text added: "SafePulse High Voltage Geiger Muller Power Supply Ver 2.0.0 02 Nov 2025"
Changed lines of the file:
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@@
+		)
+	)
+	(gr_text "SafePulse\nHigh Voltage\nGeiger Muller \nPower Supply\nVer 2.0.0\n02 Nov 2025"
+		(at 161.266 64.5414 0)
+		(layer "B.SilkS")
+		(effects
+			(font
+				(size 0.85 0.85)
+				(thickness 0.1)
+			)
+			(justify left mirror)
 		)
 	)
