File: V200/SafePulse.kicad_pcb (KiCad board)
At the start: 4 copper layers, 40.6 x 20.8 mm, 86 parts, among them IC1 S-35770E01I-K8T2U, J1 Conn_01x03_Male, J2 4208, Q1 FQT7N10L, Q2 BC846A, Q3 MMBT3906, Q4 MMBT3906, U1 TS4061AICT-1.25, U2 74HC14, U33 MAX9910EXK+T, U4 CD14538BM

Commit message: Put HV graphic back
Parts:
- added G3: LOGO, Symbol:HV warning, B.Cu at (164.0, 67.2)
Changed lines of the file:
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@@
 		)
+	)
+	(footprint "Symbol:HV warning"
+		(layer "B.Cu")
+		(at 164.0092 67.2338 180)
+		(property "Reference" "G3"
+			(at 0 0 0)
+			(layer "B.SilkS")
+			(hide yes)
+			(effects
+				(font
+					(size 1.524 1.524)
+					(thickness 0.3)
+				)
+				(justify mirror)
+			)
+		)
+		(property "Value" "LOGO"
+			(at 0.75 0 0)
+			(layer "B.SilkS")
+			(hide yes)
+			(effects
+				(font
+					(size 1.524 1.524)
+					(thickness 0.3)
+				)
+				(justify mirror)
+			)
+		)
+		(property "Datasheet" ""
+			(at 0 0 0)
+			(layer "B.Fab")
+			(hide yes)
+			(effects
+				(font
+					(size 1.27 1.27)
+					(thickness 0.15)
+				)
+				(justify mirror)
+			)
+		)
+		(property "Description" ""
+			(at 0 0 0)
+			(layer "B.Fab")
+			(hide yes)
+			(effects
+				(font
+					(size 1.27 1.27)
+					(thickness 0.15)
+				)
+				(justify mirror)
+			)
+		)
+		(attr through_hole exclude_from_pos_files exclude_from_bom dnp)
+		(fp_poly
+			(pts
+				(xy 0.125073 0.537841) (xy 0.09602 0.470411) (xy 0.05768 0.381191) (xy 0.023168 0.300728) (xy -0.021595 0.197416)
+				(xy -0.070454 0.08638) (xy -0.102569 0.014488) (xy -0.133207 -0.058041) (xy -0.152802 -0.113552)
+				(xy -0.157122 -0.138526) (xy -0.135662 -0.134844) (xy -0.082675 -0.111723) (xy -0.006547 -0.073123)
+				(xy 0.069379 -0.031507) (xy 0.158382 0.017011) (xy 0.231186 0.053353) (xy 0.279453 0.073574) (xy 0.294944 0.075186)
+				(xy 0.291077 0.048409) (xy 0.27687 -0.01591) (xy 0.254044 -0.110648) (xy 0.224322 -0.22868) (xy 0.189426 -0.362884)
+				(xy 0.185082 -0.379322) (xy 0.149353 -0.515414) (xy 0.118105 -0.636559) (xy 0.093161 -0.735517)
+				(xy 0.076342 -0.80505) (xy 0.069469 -0.837918) (xy 0.069399 -0.838976) (xy 0.083445 -0.845348) (xy 0.104657 -0.832323)
+				(xy 0.141455 -0.809158) (xy 0.152487 -0.820335) (xy 0.138678 -0.862408) (xy 0.100951 -0.931926)
+				(xy 0.061226 -0.994441) (xy 0.011063 -1.068263) (xy -0.029197 -1.124502) (xy -0.053051 -1.154189)
+				(xy -0.056377 -1.156649) (xy -0.065604 -1.135978) (xy -0.07958 -1.082377) (xy -0.092033 -1.023634)
+				(xy -0.114391 -0.908517) (xy -0.128597 -0.832091) (xy -0.135245 -0.787617) (xy -0.134931 -0.768356)
+				(xy -0.128248 -0.767568) (xy -0.115792 -0.778513) (xy -0.113476 -0.780738) (xy -0.0802 -0.80552)
+				(xy -0.068071 -0.809654) (xy -0.059089 -0.788354) (xy -0.046774 -0.731296) (xy -0.032528 -0.648749)
+				(xy -0.017753 -0.550977) (xy -0.003851 -0.448247) (xy 0.007775 -0.350825) (xy 0.015724 -0.268977)
+				(xy 0.018593 -0.212971) (xy 0.016093 -0.193446) (xy -0.008572 -0.198201) (xy -0.063297 -0.222388)
+				(xy -0.138528 -0.261538) (xy -0.182825 -0.286468) (xy -0.287281 -0.344896) (xy -0.35738 -0.379073)
+				(xy -0.39736 -0.390262) (xy -0.411458 -0.379723) (xy -0.40555 -0.352778) (xy -0.392463 -0.312767)
+				(xy -0.371236 -0.241112) (xy -0.345693 -0.150859) (xy -0.335998 -0.115665) (xy -0.30681 -0.009297)
+				(xy -0.270491 0.122492) (xy -0.232323 0.260551) (xy -0.206751 0.352778) (xy -0.131262 0.62459) (xy 0.162552 0.62459)
+			)
+			(stroke
+				(width 0)
+				(type solid)
+			)
+			(fill yes)
+			(layer "B.SilkS")
+		)
+		(fp_poly
+			(pts
+				(xy 0.103526 1.521238) (xy 0.112994 1.51659) (xy 0.129812 1.507933) (xy 0.145065 1.498624) (xy 0.16088 1.485258)
+				(xy 0.179388 1.464424) (xy 0.202715 1.432717) (xy 0.232991 1.386727) (xy 0.272343 1.323046) (xy 0.3229 1.238267)
+				(xy 0.386791 1.128982) (xy 0.466143 0.991782) (xy 0.563086 0.82326) (xy 0.679747 0.620008) (xy 0.756752 0.485792)
+				(xy 0.870014 0.288461) (xy 0.994071 0.072433) (xy 1.122313 -0.150788) (xy 1.24813 -0.369699) (xy 1.364912 -0.572797)
+				(xy 1.466049 -0.748579) (xy 1.476342 -0.76646) (xy 1.563194 -0.919331) (xy 1.640974 -1.060103) (xy 1.70683 -1.183314)
+				(xy 1.757907 -1.283502) (xy 1.79135 -1.355204) (xy 1.804305 -1.392958) (xy 1.804371 -1.394271) (xy 1.789864 -1.455043)
+				(xy 1.76016 -1.506864) (xy 1.715949 -1.561476) (xy 0.320133 -1.563178) (xy 0.059908 -1.563265) (xy -0.194568 -1.562914)
+				(xy -0.438109 -1.562159) (xy -0.665528 -1.561035) (xy -0.871637 -1.559579) (xy -1.051252 -1.557827)
+				(xy -1.199183 -1.555812) (xy -1.310246 -1.553572) (xy -1.369708 -1.551612) (xy -1.493622 -1.545249)
+				(xy -1.579595 -1.538305) (xy -1.635947 -1.529274) (xy -1.670993 -1.516649) (xy -1.693052 -1.498927)
+				(xy -1.698618 -1.492077) (xy -1.726778 -1.431622) (xy -1.734237 -1.387101) (xy -1.72319 -1.350071)
+				(xy -1.703546 -1.305916) (xy -1.434244 -1.305916) (xy -1.411759 -1.308123) (xy -1.346895 -1.310208)
+				(xy -1.243537 -1.312137) (xy -1.105574 -1.313877) (xy -0.93689 -1.315394) (xy -0.741374 -1.316655)
+				(xy -0.522911 -1.317626) (xy -0.285387 -1.318274) (xy -0.032691 -1.318566) (xy 0.034699 -1.318579)
+				(xy 0.29069 -1.318418) (xy 0.532513 -1.317952) (xy 0.756281 -1.31721) (xy 0.958109 -1.316219) (xy 1.134109 -1.315008)
+				(xy 1.280395 -1.313604) (xy 1.393081 -1.312035) (xy 1.46828 -1.310329) (xy 1.502105 -1.308515) (xy 1.503643 -1.308031)
+				(xy 1.492785 -1.284122) (xy 1.464541 -1.232515) (xy 1.431259 -1.175016) (xy 1.406166 -1.131963)
+				(xy 1.360469 -1.052929) (xy 1.296563 -0.942077) (xy 1.216842 -0.803572) (xy 1.1237 -0.641577) (xy 1.019533 -0.460255)
+				(xy 0.906735 -0.263772) (xy 0.7877 -0.05629) (xy 0.722259 0.057832) (xy 0.579769 0.306375) (xy 0.458548 0.517789)
+				(xy 0.356832 0.695071) (xy 0.272855 0.841215) (xy 0.204851 0.959219) (xy 0.151057 1.052076) (xy 0.109706 1.122784)
+				(xy 0.079033 1.174338) (xy 0.057274 1.209733) (xy 0.042662 1.231965) (xy 0.033434 1.244031) (xy 0.027823 1.248925)
+				(xy 0.024065 1.249643) (xy 0.020394 1.249181) (xy 0.020272 1.24918) (xy 0.005653 1.22982) (xy -0.028836 1.174927)
+				(xy -0.080369 1.089283) (xy -0.146118 0.977671) (xy -0.223254 0.844872) (xy -0.308949 0.69567) (xy -0.359335 0.60724)
+				(xy -0.538868 0.291042) (xy -0.705004 -0.002015) (xy -0.856739 -0.270141) (xy -0.993066 -0.511547)
+				(xy -1.112982 -0.724445) (xy -1.215481 -0.907045) (xy -1.299558 -1.057559) (xy -1.364207 -1.174197)
+				(xy -1.408424 -1.255172) (xy -1.431204 -1.298693) (xy -1.434244 -1.305916) (xy -1.703546 -1.305916)
+				(xy -1.691492 -1.27882) (xy -1.641992 -1.178981) (xy -1.577535 -1.05619) (xy -1.500969 -0.916078)
+				(xy -1.453727 -0.83191) (xy -1.354016 -0.655889) (xy -1.240156 -0.454887) (xy -1.1208 -0.244177)
+				(xy -1.004599 -0.039035) (xy -0.900206 0.145265) (xy -0.884214 0.173497) (xy -0.802669 0.317433)
+				(xy -0.7263 0.452177) (xy -0.658826 0.571172) (xy -0.603966 0.66786) (xy -0.565438 0.735684) (xy -0.549658 0.763388)
+				(xy -0.520572 0.814515) (xy -0.474849 0.895185) (xy -0.418577 0.994641) (xy -0.357848 1.102127)
+				(xy -0.353187 1.110382) (xy -0.291767 1.217355) (xy -0.233185 1.316137) (xy -0.183783 1.396241)
+				(xy -0.149902 1.44718) (xy -0.14804 1.449696) (xy -0.073945 1.516835) (xy 0.012073 1.541236)
+			)
+			(stroke
+				(width 0)
+				(type solid)
+			)
+			(fill yes)
+			(layer "B.SilkS")
+		)
+		(embedded_fonts no)
 	)
 	(footprint "TestPoint:TestPoint_Pad_1.0x1.0mm"
