File: V200/SafePulse.kicad_sch (KiCad schematic)
At the start: 89 parts, among them IC1 S-35770E01I-K8T2U, J1 Conn_01x03_Male, J2 JST SM04B-SRSS-TB(LF)(SN), Q1 FQT7N10L, Q2 BC846A, Q3 MMBT3906, Q4 MMBT3906, U1 TS4061AICT-1.25, U2 74HC14, U33 MAX9910EXK+T, U4 CD14538BM

Commit message: Updated with Allan new files
Parts:
- added R2: 10M, Resistor_SMD:R_1206_3216Metric, symbol Device:R
- H2: value Anode -> LND712
- H4: value Anode -> LND7317
Connections:
- net at C18.2, D9.2 (A), D9.3 (K)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: now also R2.1
- net at H4.1, R1.2: no longer H2.1
- new net: H2.1, R2.2
Other:
- note added: "Anode"
- moved on the sheet: R1

Commit message: V2.0.0 updated files
Parts:
- removed C20: 100pF, Capacitor_SMD:C_0805_2012Metric, symbol Device:C
- removed C21: 0.1uF, Capacitor_SMD:C_0805_2012Metric, symbol Device:C
- removed R2: 10M, Resistor_SMD:R_1206_3216Metric, symbol Device:R
- removed R26: 22M, Resistor_SMD:R_0805_2012Metric, symbol Device:R
- C1: value 110pF -> 150pF; Digikey 3372-0805B101K101BDTR-ND -> 732-12190-1-ND; LCSC C17694684 -> C520084; LCSC Part # C17694684 -> C520084
- C22: value 390pF -> 1.5nF; LCSC C1741 -> C1717; LCSC Part # C1741 -> C1717
- C4: value 47uF -> 10uF; LCSC C76636 -> C1713; LCSC Part # C76636 -> C1713
- H1, J1, two_pinheader1: now in the parts list
- H2: value LND712 -> Anode; now in the parts list
- H4: value LND7317 -> Anode; now in the parts list
- J2: value JST SM04B-SRSS-TB(LF)(SN) -> 4208; LCSC Part # C160404 -> (none)
- R17: LCSC C17721 -> C317482; LCSC Part # C17721 -> C317482
- R22: value 20K -> 12K; LCSC C2988970 -> C17444; LCSC Part # C2988970 -> C17444
- R24: value 33k -> 22k; Digikey A129767CT-ND -> CR0805-FX-2202ELFCT-ND; LCSC C17633 -> C352242; LCSC Part # C17633 -> C352242
Connections:
- net +3V3: no longer IC1.1 (~RST)
- net GND: now also C3.2, U4.1 (VSS), U4.11 (Clk-), U4.13 (R), U4.15 (VSS); no longer U4.12 (Clk+), U4.14 (RxCx)
- net at C23.1, R12.2, R6.1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: now also U4.12 (Clk+); no longer U4.11 (Clk-), U4.13 (R)
- net at H4.1, R1.2: now also H2.1
- no-connect marks 3 -> 0
Other:
- note removed: "Anode"
- moved on the sheet: D2, IC1, J2, R1, R12, R23, R24, U33, U4A, U4B
